Commit message: Code cleanup, sim in working state

File: src/es165_moveit/urdf/es165_macro.xacro (robot description, xacro)
@@ -1,5 +1,7 @@
 <?xml version="1.0"?>
-<robot xmlns:xacro="http://ros.org/wiki/xacro" name="es165d">
-  <xacro:macro name="es165_moveit" params="prefix joint_velocities_file">
+<!-- Sourced from es165 github repo
+Mesh paths updated to reflect the ROS2 build structure-->
+<robot xmlns:xacro="http://ros.org/wiki/xacro">
+  <xacro:macro name="motoman_es165" params="prefix joint_velocities_file">
     <!-- link list -->
     <link name="${prefix}base_link">
@@ -7,5 +9,5 @@
         <origin xyz="0 0 0" rpy="0 0 0"/>
           <geometry>
-            <mesh filename="package://es165_moveit/meshes/base_link.stl"/>
+            <mesh filename="package://es165_moveit/visual_meshes/base_link.stl"/>
           </geometry>
           <material name="blue">
@@ -15,5 +17,5 @@
       <collision>
         <geometry>
-          <mesh filename="package://es165_moveit/meshes/base_link.stl"/>
+          <mesh filename="package://es165_moveit/collision_meshes/base_link.stl"/>
         </geometry>
         <material name="yellow">
@@ -26,12 +28,12 @@
         <origin xyz="0 0 0" rpy="0 0 0"/>
         <geometry>
-          <mesh filename="package://es165_moveit/meshes/link_s.stl"/>
-        </geometry>
-        <material name="blue"/>
-      </visual>
-      <collision>
-        <origin xyz="0 0 0" rpy="0 0 0"/>
-        <geometry>
-          <mesh filename="package://es165_moveit/meshes/link_s.stl"/>
+          <mesh filename="package://es165_moveit/visual_meshes/link_s.stl"/>
+        </geometry>
+        <material name="blue"/>
+      </visual>
+      <collision>
+        <origin xyz="0 0 0" rpy="0 0 0"/>
+        <geometry>
+          <mesh filename="package://es165_moveit/collision_meshes/link_s.stl"/>
         </geometry>
         <material name="yellow"/>
@@ -42,12 +44,12 @@
         <origin xyz="0 0 0" rpy="0 0 0"/>
         <geometry>
-          <mesh filename="package://es165_moveit/meshes/link_l.stl"/>
-        </geometry>
-        <material name="blue"/>
-      </visual>
-      <collision>
-        <origin xyz="0 0 0" rpy="0 0 0"/>
-        <geometry>
-          <mesh filename="package://es165_moveit/meshes/link_l.stl"/>
+          <mesh filename="package://es165_moveit/visual_meshes/link_l.stl"/>
+        </geometry>
+        <material name="blue"/>
+      </visual>
+      <collision>
+        <origin xyz="0 0 0" rpy="0 0 0"/>
+        <geometry>
+          <mesh filename="package://es165_moveit/collision_meshes/link_l.stl"/>
         </geometry>
         <material name="yellow"/>
@@ -58,12 +60,12 @@
         <origin xyz="0 0 0" rpy="0 0 0"/>
         <geometry>
-          <mesh filename="package://es165_moveit/meshes/link_u.stl"/>
-        </geometry>
-        <material name="blue"/>
-      </visual>
-      <collision>
-        <origin xyz="0 0 0" rpy="0 0 0"/>
-        <geometry>
-          <mesh filename="package://es165_moveit/meshes/link_u.stl"/>
+          <mesh filename="package://es165_moveit/visual_meshes/link_u.stl"/>
+        </geometry>
+        <material name="blue"/>
+      </visual>
+      <collision>
+        <origin xyz="0 0 0" rpy="0 0 0"/>
+        <geometry>
+          <mesh filename="package://es165_moveit/collision_meshes/link_u.stl"/>
         </geometry>
         <material name="yellow"/>
@@ -74,5 +76,5 @@
         <origin xyz="0 0 0" rpy="0 0 0"/>
       <geometry>
-        <mesh filename="package://es165_moveit/meshes/link_r.stl"/>
+        <mesh filename="package://es165_moveit/visual_meshes/link_r.stl"/>
       </geometry>
       <material name="blue"/>
@@ -81,5 +83,5 @@
         <origin xyz="0 0 0" rpy="0 0 0"/>
         <geometry>
-          <mesh filename="package://es165_moveit/meshes/link_r.stl"/>
+          <mesh filename="package://es165_moveit/collision_meshes/link_r.stl"/>
         </geometry>
         <material name="yellow"/>
@@ -90,12 +92,12 @@
         <origin xyz="0 0 0" rpy="0 0 0"/>
         <geometry>
-          <mesh filename="package://es165_moveit/meshes/link_b.stl"/>
-        </geometry>
-        <material name="blue"/>
-      </visual>
-      <collision>
-        <origin xyz="0 0 0" rpy="0 0 0"/>
-        <geometry>
-          <mesh filename="package://es165_moveit/meshes/link_b.stl"/>
+          <mesh filename="package://es165_moveit/visual_meshes/link_b.stl"/>
+        </geometry>
+        <material name="blue"/>
+      </visual>
+      <collision>
+        <origin xyz="0 0 0" rpy="0 0 0"/>
+        <geometry>
+          <mesh filename="package://es165_moveit/collision_meshes/link_b.stl"/>
         </geometry>
         <material name="yellow"/>
@@ -106,5 +108,5 @@
         <origin xyz="0 0 0" rpy="0 0 0"/>
           <geometry>
-            <mesh filename="package://es165_moveit/meshes/link_t.stl"/>
+            <mesh filename="package://es165_moveit/visual_meshes/link_t.stl"/>
           </geometry>
           <material name="black">
@@ -115,10 +117,9 @@
         <origin xyz="0 0 0" rpy="0 0 0"/>
         <geometry>
-          <mesh filename="package://es165_moveit/meshes/link_t.stl"/>
+          <mesh filename="package://es165_moveit/collision_meshes/link_t.stl"/>
         </geometry>
         <material name="black"/>
       </collision>
     </link>
-    <link name="${prefix}tool0"/>
     <!--
       Balancer and rod are disabled as without a mimic joint they will not update
@@ -130,12 +131,12 @@
         <origin xyz="0 0 0" rpy="0 0 0"/>
         <geometry>
-          <mesh filename="package://es165_moveit/meshes/balancer_piston.stl"/>
-        </geometry>
-        <material name="blue"/>
-      </visual>
-      <collision>
-        <origin xyz="0 0 0" rpy="0 0 0"/>
-        <geometry>
-          <mesh filename="package://es165_moveit/meshes/balancer_piston.stl"/>
+          <mesh filename="package://es165_moveit/balancer_piston.stl"/>
+        </geometry>
+        <material name="blue"/>
+      </visual>
+      <collision>
+        <origin xyz="0 0 0" rpy="0 0 0"/>
+        <geometry>
+          <mesh filename="package://es165_moveit/collision/balancer_piston.stl"/>
         </geometry>
         <material name="yellow"/>
@@ -146,5 +147,5 @@
         <origin xyz="0 0 0" rpy="0 0 0"/>
         <geometry>
-          <mesh filename="package://es165_moveit/meshes/balancer_rod.stl"/>
+          <mesh filename="package://es165_moveit/balancer_rod.stl"/>
         </geometry>
         <material name="blue">
@@ -155,5 +156,5 @@
         <origin xyz="0 0 0" rpy="0 0 0"/>
         <geometry>
-          <mesh filename="package://es165_moveit/meshes/balancer_rod.stl"/>
+          <mesh filename="package://es165_moveit/collision/balancer_rod.stl"/>
         </geometry>
         <material name="yellow"/>
@@ -206,9 +207,4 @@
       <limit lower="${radians(-360)}" upper="${radians(360)}" effort="0" velocity="${radians(velocities['joint_6_t'])}"/>
     </joint>
-    <joint name="${prefix}joint_t-tool0" type="fixed">
-      <origin xyz="0 0 0" rpy="0 ${pi} 0"/>
-      <parent link="${prefix}link_t"/>
-      <child link="${prefix}tool0"/>
-    </joint>
     <!--
       See earlier comment about balancer and piston.
@@ -232,5 +228,18 @@
       <child link="${prefix}base"/>
     </joint>
+    <!-- ROS-Industrial 'flange' frame: attachment point for EEF models -->
+    <link name="${prefix}flange"/>
+    <joint name="${prefix}link_t-flange" type="fixed">
+      <origin xyz="0 0 0" rpy="0 ${radians(90)} 0"/>
+      <parent link="${prefix}link_t"/>
+      <child link="${prefix}flange"/>
+    </joint>
+    <!-- ROS-Industrial 'tool0' frame: all-zeros tool frame -->
+    <link name="${prefix}tool0"/>
+    <joint name="${prefix}flange-tool0" type="fixed">
+      <origin xyz="0 0 0" rpy="${radians(180)} ${radians(-90)} 0"/>
+      <parent link="${prefix}flange"/>
+      <child link="${prefix}tool0"/>
+    </joint>
   </xacro:macro>
-  <!-- <xacro:es165_moveit prefix="" joint_velocities_file="$(find es165_moveit)/config/joint_velocities_dx100.yaml"/> -->
 </robot>

File: src/es165_moveit/urdf/es_165.ros2_control.xacro (robot description, xacro)
@@ -3,56 +3,96 @@
   <xacro:macro name="es165_ros2_control" params="name">
     <!-- ROS 2 control block -->
-    <ros2_control name="arm_controller" type="system">
+    <ros2_control name="es165_arm" type="system">
       <!-- Isaac Sim hardware interface -->
       <hardware>
-      <!-- This plugin name must match the Isaac ROS control plugin -->
-        <!-- <plugin>topic_based_ros2_control/TopicBasedSystem</plugin>
+        <!-- Using topic_based_ros2_control for Isaac Sim integration -->
+        <plugin>topic_based_ros2_control/TopicBasedSystem</plugin>
         <param name="joint_commands_topic">isaac_joint_commands</param>
-        <param name="joint_states_topic">isaac_joint_states</param> -->
-        <plugin>mock_components/GenericSystem</plugin>
-        <!-- <param name="fake_sensor_commands">true</param> -->
+        <param name="joint_states_topic">isaac_joint_states</param>
       </hardware>
       <!-- Joint interfaces -->
       <joint name="joint_1_s">
-        <command_interface name="position"/>
-        <state_interface name="position"/>
-        <state_interface name="velocity"/>
-        <state_interface name="effort"/>
-        <!-- <state_interface name="effort"/> -->
+        <command_interface name="position">
+          <param name="initial_value">0.0</param>
+        </command_interface>
+        <state_interface name="position">
+          <param name="initial_value">0.0</param>
+        </state_interface>
+        <state_interface name="velocity">
+          <param name="initial_value">0.0</param>
+        </state_interface>
+        <state_interface name="effort">
+          <param name="initial_value">0.0</param>
+        </state_interface>
       </joint>
       <joint name="joint_2_l">
-        <command_interface name="position"/>
-        <state_interface name="position"/>
-        <state_interface name="velocity"/>
-        <state_interface name="effort"/>
-        <!-- <state_interface name="effort"/> -->
+        <command_interface name="position">
+          <param name="initial_value">0.0</param>
+        </command_interface>
+        <state_interface name="position">
+          <param name="initial_value">0.0</param>
+        </state_interface>
+        <state_interface name="velocity">
+          <param name="initial_value">0.0</param>
+        </state_interface>
+        <state_interface name="effort">
+          <param name="initial_value">0.0</param>
+        </state_interface>
       </joint>
       <joint name="joint_3_u">
-        <command_interface name="position"/>
-        <state_interface name="position"/>
-        <state_interface name="velocity"/>
-        <state_interface name="effort"/>
-        <!-- <state_interface name="effort"/> -->
+        <command_interface name="position">
+          <param name="initial_value">0.0</param>
+        </command_interface>
+        <state_interface name="position">
+          <param name="initial_value">0.0</param>
+        </state_interface>
+        <state_interface name="velocity">
+          <param name="initial_value">0.0</param>
+        </state_interface>
+        <state_interface name="effort">
+          <param name="initial_value">0.0</param>
+        </state_interface>
       </joint>
       <joint name="joint_4_r">
-        <command_interface name="position"/>
-        <state_interface name="position"/>
-        <state_interface name="velocity"/>
-        <state_interface name="effort"/>
-        <!-- <state_interface name="effort"/> -->
+        <command_interface name="position">
+          <param name="initial_value">0.0</param>
+        </command_interface>
+        <state_interface name="position">
+          <param name="initial_value">0.0</param>
+        </state_interface>
+        <state_interface name="velocity">
+          <param name="initial_value">0.0</param>
+        </state_interface>
+        <state_interface name="effort">
+          <param name="initial_value">0.0</param>
+        </state_interface>
       </joint>
       <joint name="joint_5_b">
-        <command_interface name="position"/>
-        <state_interface name="position"/>
-        <state_interface name="velocity"/>
-        <state_interface name="effort"/>
-        <!-- <state_interface name="effort"/> -->
+        <command_interface name="position">
+          <param name="initial_value">0.0</param>
+        </command_interface>
+        <state_interface name="position">
+          <param name="initial_value">0.0</param>
+        </state_interface>
+        <state_interface name="velocity">
+          <param name="initial_value">0.0</param>
+        </state_interface>
+        <state_interface name="effort">
+          <param name="initial_value">0.0</param>
+        </state_interface>
       </joint>
       <joint name="joint_6_t">
-        <command_interface name="position"/>
-        <state_interface name="position"/>
-        <state_interface name="velocity"/>
-        <state_interface name="effort"/>
-        <!-- <state_interface name="effort"/> -->
+        <command_interface name="position">
+          <param name="initial_value">0.0</param>
+        </command_interface>
+        <state_interface name="position">
+          <param name="initial_value">0.0</param>
+        </state_interface>
+        <state_interface name="velocity">
+          <param name="initial_value">0.0</param>
+        </state_interface>
+        <state_interface name="effort">
+          <param name="initial_value">0.0</param>
+        </state_interface>
       </joint>
     </ros2_control>

File: src/es165_moveit_moveit_config/config/es165.xacro (robot description, xacro)
@@ -1,3 +1,4 @@
 <?xml version="1.0" ?>
+<!-- Defines references and sets up the main xacro and ros2 controllers -->
 <robot name="es165d" xmlns:xacro="http://ros.org/wiki/xacro">
   <xacro:arg name="joint_velocities_file" default="$(find es165_moveit)/config/joint_velocities_dx100.yaml"/>
@@ -5,6 +6,6 @@
   <!-- ros2 control setup -->
   <xacro:include filename="$(find es165_moveit)/urdf/es_165.ros2_control.xacro" />
-  <xacro:es165_ros2_control name="arm_controller"/>
+  <xacro:es165_ros2_control name="es165_arm"/>
   <!---->
-  <xacro:es165_moveit prefix="" joint_velocities_file="$(arg joint_velocities_file)"/>
+  <xacro:motoman_es165 prefix="" joint_velocities_file="$(arg joint_velocities_file)"/>
 </robot>
