Commit message: servo update, usd/urdf files too large for commit, control using rw speed change (torque) as an option

File: src/es165_moveit/urdf/es165_macro.xacro (robot description, xacro)
@@ -4,4 +4,8 @@
     <!-- link list -->
     <link name="${prefix}base_link">
+      <inertial>
+        <mass value="305"/>
+        <inertia ixx="1" ixy="0" ixz="0" iyy="1" iyz="0" izz="1"/>
+      </inertial>
       <visual>
         <origin xyz="0 0 0" rpy="0 0 0"/>
@@ -23,4 +27,8 @@
     </link>
     <link name="${prefix}link_s">
+      <inertial>
+        <mass value="422.18"/>
+        <inertia ixx="14.17" iyy="38.48" izz="40.88" ixy="0" ixz="0" iyz="0"/>
+      </inertial>
       <visual>
         <origin xyz="0 0 0" rpy="0 0 0"/>
@@ -39,4 +47,8 @@
     </link>
     <link name="${prefix}link_l">
+      <inertial>
+        <mass value="259.5"/>
+        <inertia ixx="3.57" iyy="31.35" izz="32.24" ixy="0" ixz="0" iyz="0"/>
+      </inertial>
       <visual>
         <origin xyz="0 0 0" rpy="0 0 0"/>
@@ -55,4 +67,8 @@
     </link>
     <link name="${prefix}link_u">
+      <inertial>
+        <mass value="258.7"/>
+        <inertia ixx="5.59" iyy="25.03" izz="27.08" ixy="0" ixz="0" iyz="0"/>
+      </inertial>
       <visual>
         <origin xyz="0 0 0" rpy="0 0 0"/>
@@ -71,4 +87,8 @@
     </link>
     <link name="${prefix}link_r">
+      <inertial>
+        <mass value="13.02"/>
+        <inertia ixx="0.03" iyy="0.1" izz="0.1" ixy="0" ixz="0" iyz="0"/>
+      </inertial>
       <visual>
         <origin xyz="0 0 0" rpy="0 0 0"/>
@@ -87,4 +107,8 @@
     </link>
     <link name="${prefix}link_b">
+      <inertial>
+        <mass value="27.436"/>
+        <inertia ixx="0.19" iyy="0.28" izz="0.35" ixy="0" ixz="0" iyz="0"/>
+      </inertial>
       <visual>
         <origin xyz="0 0 0" rpy="0 0 0"/>
@@ -103,4 +127,8 @@
     </link>
     <link name="${prefix}link_t">
+      <inertial>
+        <mass value="2.16"/>
+        <inertia ixx="0.001" iyy="0.001" izz="0.01" ixy="0" ixz="0" iyz="0"/>
+      </inertial>
       <visual>
         <origin xyz="0 0 0" rpy="0 0 0"/>
@@ -118,4 +146,97 @@
         </geometry>
         <material name="black"/>
+      </collision>
+    </link>
+    <link name="${prefix}ee_base_link">
+      <inertial>
+        <mass value="30.24"/>
+        <inertia ixx="0.669" iyy="2.609" izz="3.261" ixy="0" ixz="0" iyz="0"/>
+      </inertial>
+      <visual>
+        <origin xyz="0 0 0" rpy="0 0 0"/>
+        <geometry>
+          <mesh filename="package://es165_moveit/visual_meshes/ee_base_link.stl"/>
+        </geometry>
+        <material name="grey">
+          <color rgba="0.7 0.7 0.7 1"/>
+        </material>
+      </visual>
+      <collision>
+        <origin xyz="0 0 0" rpy="0 0 0"/>
+        <geometry>
+          <mesh filename="package://es165_moveit/collision_meshes/ee_base_link.stl"/>
+        </geometry>
+      </collision>
+    </link>
+    <link name="${prefix}rw1">
+      <inertial>
+        <mass value="0.490"/>
+        <inertia izz="0.0003" ixx="0.001" iyy="0.001" ixy="0" ixz="0" iyz="0"/>
+      </inertial>
+      <visual>
+        <origin rpy="0.00000 0.00000 0.00000" xyz="0.00000 0.00000 0.00000"/>
+        <geometry>
+          <mesh filename="package://es165_moveit/urdf/rw1_visual.stl" scale="1.00000 1.00000 1.00000"/>
+        </geometry>
+      </visual>
+      <collision>
+        <origin rpy="0.00000 0.00000 0.00000" xyz="0.00000 0.00000 0.00000"/>
+        <geometry>
+          <mesh filename="package://es165_moveit/urdf/rw1_collision.stl" scale="1.00000 1.00000 1.00000"/>
+        </geometry>
+      </collision>
+    </link>
+    <link name="${prefix}rw2">
+      <inertial>
+        <mass value="0.490"/>
+        <inertia izz="0.0003" ixx="0.001" iyy="0.001" ixy="0" ixz="0" iyz="0"/>
+      </inertial>
+      <visual>
+        <origin rpy="0.00000 0.00000 0.00000" xyz="0.00000 0.00000 0.00000"/>
+        <geometry>
+          <mesh filename="package://es165_moveit/urdf/rw2_visual.stl" scale="1.00000 1.00000 1.00000"/>
+        </geometry>
+      </visual>
+      <collision>
+        <origin rpy="0.00000 0.00000 0.00000" xyz="0.00000 0.00000 0.00000"/>
+        <geometry>
+          <mesh filename="package://es165_moveit/urdf/rw2_collision.stl" scale="1.00000 1.00000 1.00000"/>
+        </geometry>
+      </collision>
+    </link>
+    <link name="${prefix}rw3">
+      <inertial>
+        <mass value="0.490"/>
+        <inertia izz="0.0003" ixx="0.001" iyy="0.001" ixy="0" ixz="0" iyz="0"/>
+      </inertial>
+      <visual>
+        <origin rpy="0.00000 0.00000 0.00000" xyz="0.00000 0.00000 0.00000"/>
+        <geometry>
+          <mesh filename="package://es165_moveit/urdf/rw3_visual.stl" scale="1.00000 1.00000 1.00000"/>
+        </geometry>
+      </visual>
+      <collision>
+        <origin rpy="0.00000 0.00000 0.00000" xyz="0.00000 0.00000 0.00000"/>
+        <geometry>
+          <mesh filename="package://es165_moveit/urdf/rw3_collision.stl" scale="1.00000 1.00000 1.00000"/>
+        </geometry>
+      </collision>
+    </link>
+    <link name="${prefix}rw4">
+      <inertial>
+        <mass value="0.490"/>
+        <inertia izz="0.0003" ixx="0.001" iyy="0.001" ixy="0" ixz="0" iyz="0"/>
+      </inertial>
+      <visual>
+        <origin rpy="0.00000 0.00000 0.00000" xyz="0.00000 0.00000 0.00000"/>
+        <geometry>
+          <mesh filename="package://es165_moveit/urdf/rw4_visual.stl" scale="1.00000 1.00000 1.00000"/>
+        </geometry>
+      </visual>
+      <collision>
+        <origin rpy="0.00000 0.00000 0.00000" xyz="0.00000 0.00000 0.00000"/>
+        <geometry>
+          <mesh filename="package://es165_moveit/urdf/rw4_collision.stl" scale="1.00000 1.00000 1.00000"/>
+        </geometry>
       </collision>
     </link>
@@ -205,4 +326,33 @@
       <limit lower="${radians(-360)}" upper="${radians(360)}" effort="0" velocity="${radians(velocities['joint_6_t'])}"/>
     </joint>
+    <joint name="ee_base_link_joint" type="fixed">
+      <origin xyz="0.004513 0 -0.0745" rpy="1.570796 0 0" />
+      <parent link="link_t" />
+      <child link="ee_base_link" />
+    </joint>
+    <joint name="${prefix}rw1_joint" type="continuous">
+      <origin xyz="0.000974 -0.055246 0.001299" rpy="1.570797 0 0" />
+      <parent link="ee_base_link" />
+      <child link="rw1" />
+      <axis xyz="0 0 1" />
+    </joint>
+    <joint name="${prefix}rw3_joint" type="continuous">
+      <origin xyz="0.118956 -0.105533 0.001298" rpy="1.570796 0 -1.570796" />
+      <parent link="ee_base_link" />
+      <child link="rw3" />
+      <axis xyz="0 0 1" />
+    </joint>
+    <joint name="${prefix}rw2_joint" type="continuous">
+      <origin xyz="-0.127511 -0.105533 0.001298" rpy="1.570796 0 1.570796" />
+      <parent link="ee_base_link" />
+      <child link="rw2" />
+      <axis xyz="0 0 1" />
+    </joint>
+    <joint name="${prefix}rw4_joint" type="continuous">
+      <origin xyz="0.000974 -0.115515 0.131297" rpy="3.141592 0 0" />
+      <parent link="ee_base_link" />
+      <child link="rw4" />
+      <axis xyz="0 0 1" />
+    </joint>
     <!--
       See earlier comment about balancer and piston.
@@ -240,4 +390,5 @@
       <child link="${prefix}tool0"/>
     </joint>
+    <!-- End Effector attached to tool0 -->
   </xacro:macro>
 </robot>

File: src/es165_moveit/urdf/es_165.ros2_control.xacro (robot description, xacro)
@@ -25,7 +25,4 @@
           <param name="initial_value">0.0</param>
         </state_interface>
-        <state_interface name="effort">
-          <param name="initial_value">0.0</param>
-        </state_interface>
       </joint>
       <joint name="joint_2_l">
@@ -40,7 +37,4 @@
         </state_interface>
         <state_interface name="velocity">
-          <param name="initial_value">0.0</param>
-        </state_interface>
-        <state_interface name="effort">
           <param name="initial_value">0.0</param>
         </state_interface>
@@ -59,7 +53,4 @@
           <param name="initial_value">0.0</param>
         </state_interface>
-        <state_interface name="effort">
-          <param name="initial_value">0.0</param>
-        </state_interface>
       </joint>
       <joint name="joint_4_r">
@@ -74,7 +65,4 @@
         </state_interface>
         <state_interface name="velocity">
-          <param name="initial_value">0.0</param>
-        </state_interface>
-        <state_interface name="effort">
           <param name="initial_value">0.0</param>
         </state_interface>
@@ -93,7 +81,4 @@
           <param name="initial_value">0.0</param>
         </state_interface>
-        <state_interface name="effort">
-          <param name="initial_value">0.0</param>
-        </state_interface>
       </joint>
       <joint name="joint_6_t">
@@ -110,8 +95,62 @@
           <param name="initial_value">0.0</param>
         </state_interface>
-        <state_interface name="effort">
-          <param name="initial_value">0.0</param>
-        </state_interface>
       </joint>
+    <!-- RW joints-->
+    <joint name="rw1_joint">
+      <command_interface name="position">
+        <param name="initial_value">0.0</param>
+      </command_interface>
+      <command_interface name="velocity">
+        <param name="initial_value">0.0</param>
+      </command_interface>
+      <state_interface name="position">
+        <param name="initial_value">0.0</param>
+      </state_interface>
+      <state_interface name="velocity">
+        <param name="initial_value">0.0</param>
+      </state_interface>
+    </joint>
+    <joint name="rw3_joint">
+      <command_interface name="position">
+        <param name="initial_value">0.0</param>
+      </command_interface>
+      <command_interface name="velocity">
+        <param name="initial_value">0.0</param>
+      </command_interface>
+      <state_interface name="position">
+        <param name="initial_value">0.0</param>
+      </state_interface>
+      <state_interface name="velocity">
+        <param name="initial_value">0.0</param>
+      </state_interface>
+    </joint>
+    <joint name="rw2_joint">
+      <command_interface name="position">
+        <param name="initial_value">0.0</param>
+      </command_interface>
+      <command_interface name="velocity">
+        <param name="initial_value">0.0</param>
+      </command_interface>
+      <state_interface name="position">
+        <param name="initial_value">0.0</param>
+      </state_interface>
+      <state_interface name="velocity">
+        <param name="initial_value">0.0</param>
+      </state_interface>
+    </joint>
+    <joint name="rw4_joint">
+      <command_interface name="position">
+        <param name="initial_value">0.0</param>
+      </command_interface>
+      <command_interface name="velocity">
+        <param name="initial_value">0.0</param>
+      </command_interface>
+      <state_interface name="position">
+        <param name="initial_value">0.0</param>
+      </state_interface>
+      <state_interface name="velocity">
+        <param name="initial_value">0.0</param>
+      </state_interface>
+    </joint>
     </ros2_control>
   </xacro:macro>

Commit message: updated with new collision meshes

File: src/es165_moveit/urdf/es165_macro.xacro (robot description, xacro)
@@ -11,5 +11,5 @@
         <origin xyz="0 0 0" rpy="0 0 0"/>
           <geometry>
-            <mesh filename="package://es165_moveit/visual_meshes/base_link.stl"/>
+            <mesh filename="package://es165_moveit/urdf/base_link_visual.stl"/>
           </geometry>
           <material name="blue">
@@ -19,5 +19,5 @@
       <collision>
         <geometry>
-          <mesh filename="package://es165_moveit/collision_meshes/base_link.stl"/>
+          <mesh filename="package://es165_moveit/urdf/base_link_collision.stl"/>
         </geometry>
         <material name="yellow">
@@ -34,12 +34,12 @@
         <origin xyz="0 0 0" rpy="0 0 0"/>
         <geometry>
-          <mesh filename="package://es165_moveit/visual_meshes/link_s.stl"/>
-        </geometry>
-        <material name="blue"/>
-      </visual>
-      <collision>
-        <origin xyz="0 0 0" rpy="0 0 0"/>
-        <geometry>
-          <mesh filename="package://es165_moveit/collision_meshes/link_s.stl"/>
+          <mesh filename="package://es165_moveit/urdf/link_s_visual.stl"/>
+        </geometry>
+        <material name="blue"/>
+      </visual>
+      <collision>
+        <origin xyz="0 0 0" rpy="0 0 0"/>
+        <geometry>
+          <mesh filename="package://es165_moveit/urdf/link_s_collision.stl"/>
         </geometry>
         <material name="yellow"/>
@@ -54,12 +54,12 @@
         <origin xyz="0 0 0" rpy="0 0 0"/>
         <geometry>
-          <mesh filename="package://es165_moveit/visual_meshes/link_l.stl"/>
-        </geometry>
-        <material name="blue"/>
-      </visual>
-      <collision>
-        <origin xyz="0 0 0" rpy="0 0 0"/>
-        <geometry>
-          <mesh filename="package://es165_moveit/collision_meshes/link_l.stl"/>
+          <mesh filename="package://es165_moveit/urdf/link_l_visual.stl"/>
+        </geometry>
+        <material name="blue"/>
+      </visual>
+      <collision>
+        <origin xyz="0 0 0" rpy="0 0 0"/>
+        <geometry>
+          <mesh filename="package://es165_moveit/urdf/link_l_collision.stl"/>
         </geometry>
         <material name="yellow"/>
@@ -74,12 +74,12 @@
         <origin xyz="0 0 0" rpy="0 0 0"/>
         <geometry>
-          <mesh filename="package://es165_moveit/visual_meshes/link_u.stl"/>
-        </geometry>
-        <material name="blue"/>
-      </visual>
-      <collision>
-        <origin xyz="0 0 0" rpy="0 0 0"/>
-        <geometry>
-          <mesh filename="package://es165_moveit/collision_meshes/link_u.stl"/>
+          <mesh filename="package://es165_moveit/urdf/link_u_visual.stl"/>
+        </geometry>
+        <material name="blue"/>
+      </visual>
+      <collision>
+        <origin xyz="0 0 0" rpy="0 0 0"/>
+        <geometry>
+          <mesh filename="package://es165_moveit/urdf/link_u_collision.stl"/>
         </geometry>
         <material name="yellow"/>
@@ -94,5 +94,5 @@
         <origin xyz="0 0 0" rpy="0 0 0"/>
       <geometry>
-        <mesh filename="package://es165_moveit/visual_meshes/link_r.stl"/>
+        <mesh filename="package://es165_moveit/urdf/link_r_visual.stl"/>
       </geometry>
       <material name="blue"/>
@@ -101,5 +101,5 @@
         <origin xyz="0 0 0" rpy="0 0 0"/>
         <geometry>
-          <mesh filename="package://es165_moveit/collision_meshes/link_r.stl"/>
+          <mesh filename="package://es165_moveit/urdf/link_r_collision.stl"/>
         </geometry>
         <material name="yellow"/>
@@ -114,12 +114,12 @@
         <origin xyz="0 0 0" rpy="0 0 0"/>
         <geometry>
-          <mesh filename="package://es165_moveit/visual_meshes/link_b.stl"/>
-        </geometry>
-        <material name="blue"/>
-      </visual>
-      <collision>
-        <origin xyz="0 0 0" rpy="0 0 0"/>
-        <geometry>
-          <mesh filename="package://es165_moveit/collision_meshes/link_b.stl"/>
+          <mesh filename="package://es165_moveit/urdf/link_b_visual.stl"/>
+        </geometry>
+        <material name="blue"/>
+      </visual>
+      <collision>
+        <origin xyz="0 0 0" rpy="0 0 0"/>
+        <geometry>
+          <mesh filename="package://es165_moveit/urdf/link_b_collision.stl"/>
         </geometry>
         <material name="yellow"/>
@@ -134,5 +134,5 @@
         <origin xyz="0 0 0" rpy="0 0 0"/>
           <geometry>
-            <mesh filename="package://es165_moveit/visual_meshes/link_t.stl"/>
+            <mesh filename="package://es165_moveit/urdf/link_t_visual.stl"/>
           </geometry>
           <material name="black">
@@ -143,5 +143,5 @@
         <origin xyz="0 0 0" rpy="0 0 0"/>
         <geometry>
-          <mesh filename="package://es165_moveit/collision_meshes/link_t.stl"/>
+          <mesh filename="package://es165_moveit/urdf/link_t_collision.stl"/>
         </geometry>
         <material name="black"/>
@@ -156,5 +156,5 @@
         <origin xyz="0 0 0" rpy="0 0 0"/>
         <geometry>
-          <mesh filename="package://es165_moveit/visual_meshes/ee_base_link.stl"/>
+          <mesh filename="package://es165_moveit/urdf/ee_base_link_visual.stl"/>
         </geometry>
         <material name="grey">
@@ -165,5 +165,5 @@
         <origin xyz="0 0 0" rpy="0 0 0"/>
         <geometry>
-          <mesh filename="package://es165_moveit/collision_meshes/ee_base_link.stl"/>
+          <mesh filename="package://es165_moveit/urdf/ee_base_link_collision.stl"/>
         </geometry>
       </collision>

Commit message: removed bloat

File: src/es165_moveit/urdf/es165_macro.xacro (robot description, xacro)
@@ -241,45 +241,4 @@
       </collision>
     </link>
-    <!--
-      Balancer and rod are disabled as without a mimic joint they will not update
-      their pose properly, leading to MoveIt detecting collisions which cannot
-      happen with the real robot (as the balancer is essentially a passive element
-      and cannot come into collision with anything due to joint limits).
-    <link name="${prefix}balancer_piston">
-      <visual>
-        <origin xyz="0 0 0" rpy="0 0 0"/>
-        <geometry>
-          <mesh filename="package://es165_moveit/balancer_piston.stl"/>
-        </geometry>
-        <material name="blue"/>
-      </visual>
-      <collision>
-        <origin xyz="0 0 0" rpy="0 0 0"/>
-        <geometry>
-          <mesh filename="package://es165_moveit/collision/balancer_piston.stl"/>
-        </geometry>
-        <material name="yellow"/>
-      </collision>
-    </link>
-    <link name="${prefix}balancer_rod">
-      <visual>
-        <origin xyz="0 0 0" rpy="0 0 0"/>
-        <geometry>
-          <mesh filename="package://es165_moveit/balancer_rod.stl"/>
-        </geometry>
-        <material name="blue">
-          <color rgba="1 1 1 1"/>
-        </material>
-      </visual>
-      <collision>
-        <origin xyz="0 0 0" rpy="0 0 0"/>
-        <geometry>
-          <mesh filename="package://es165_moveit/collision/balancer_rod.stl"/>
-        </geometry>
-        <material name="yellow"/>
-      </collision>
-    </link>
-    -->
-    <!-- end of link list -->
     <!-- joint list -->
     <xacro:property name="velocities" value="${xacro.load_yaml(joint_velocities_file)}" />
